File: hardware/v1-ornament-board/kicad/v1-ornament-board.kicad_sch (KiCad schematic)
At the start: 245 parts, among them J1 Battery_JST-PH-2.0, SW1 SKRHABE010, U1 XIAO-SAMD21-SMD, U2 74AHCT1G125, U3 MCP73832-2-OT

Commit message: Clean up V1 LED array wiring, decoupling caps, and add tooling holes
- Redraw the WS2812 daisy-chain data connections as explicit wires
  (matching the user's D12-D13-D14 example) instead of floating,
  overlapping labels, for all same-row LED pairs
- Reposition and resize all 118 decoupling caps to Device:C_Small
  using C13 as the template, editing symbols in place so PCB
  footprint links survive (no re-placement needed)
- Add two JLCPCB assembly tooling-hole placeholders (TH1/TH2) per
  their NPTH spec, for the user to position by hand
- Close a 1-micron gap in the decorative tab shape's inner lens
  outline on F.Cu so it forms a valid closed loop for zone fill

Co-Authored-By: Claude Sonnet 5 <noreply@anthropic.com>
Parts:
- C10, C100, C101, C102, C103, C104, C105, C106, C107, C108, C109, C11, C110, C111, C112, C113, C114, C115, C116, C117, C118, C119, C12, C120, C121, C122, C123, C124, C13, C14, C15, C16, C17, C18, C19, C20, C21, C22, C23, C24, C25, C26, C27, C28, C29, C30, C31, C32, C33, C34, C35, C36, C37, C38, C39, C4, C40, C41, C42, C43, C44, C45, C46, C47, C48, C49, C5, C50, C51, C52, C53, C54, C55, C56, C57, C58, C59, C60, C61, C62, C63, C64, C65, C66, C67, C68, C69, C70, C71, C72, C73, C74, C75, C76, C77, C78, C79, C80, C81, C82, C83, C84, C85, C86, C87, C88, C89, C9, C90, C91, C92, C93, C94, C95, C96, C97, C98, C99: symbol Device:C -> Device:C_Small
- D122: value STAT_LED -> KT-0603R
- R1: value 10k -> 2.49k
Connections:
- net TRIP_LED_A: no longer names the net of D124.2 (A), R3.2
Other:
- moved on the sheet: C10, C100, C101, C102, C103, C104, C105, C106, C107, C108, C109, C11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

Commit message: Move ordering docs to ignored folder; move Emulator to pages, add pixel palette
- Move digikey order/invoice into hardware/v1-ornament-board/ordering-docs/ (gitignored)
- Gitignore KiCad manual pre-edit .bak snapshots and local xmas2026.zip backup
- Rework web emulator: Emulator moves to pages/, adds Pixel/PixelPalette components and virtualHardware
- V1 board fab/KiCad updates (hand-solder BOM, footprint swap script)

Co-Authored-By: Claude Sonnet 5 <noreply@anthropic.com>
Parts:
- U3: value MCP73832-2-OT -> MCP73832-2-MC; footprint Package_TO_SOT_SMD:SOT-23-5 -> Package_DFN_QFN:DFN-8-1EP_3x2mm_P0.5mm_EP1.7x1.4mm; symbol Battery_Management:MCP73832-2-OT -> Battery_Management:MCP73832-2-MC
Connections:
- net +5V: now also U3.1 (V_{DD}), U3.2 (V_{DD}); no longer U3.4 (V_{DD})
- net GND: now also U3.6 (V_{SS}); no longer U3.2 (V_{SS})
- net JOY_DOWN: now also SW1.6, U1.2 (D1); no longer SW1.3, U1.3 (D2)
- net JOY_LEFT: now also SW1.3, U1.3 (D2); no longer SW1.4, U1.1 (D0)
- net JOY_RIGHT: now also SW1.4, U1.1 (D0); no longer SW1.6, U1.2 (D1)
- net JOY_UP: now also U1.5 (D4); no longer U1.7 (D6)
- net PROG: now also U3.8 (PROG); no longer U3.5 (PROG)
- net STAT: now also U3.5 (STAT); no longer U3.1 (STAT)
- net VBATT: now also U3.4 (V_{BAT})
Changed lines of the file:
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@@
 	)
 	(no_connect
+		(at 452.12 176.53)
+	)
+	(no_connect
 		(at 468.63 140.97)
 	)
@@
 	)
 	(no_connect
-		(at 452.12 168.91)
-	)
-	(no_connect
 		(at 495.3 176.53)
 	)
@@
 	(wire
 		(pts
-			(xy 223.52 344.17) (xy 215.9 344.17)
+			(xy 222.25 344.17) (xy 215.9 344.17)
 		)
 		(stroke
@@
 	(wire
 		(pts
+			(xy 445.77 168.91) (xy 452.12 168.91)
+		)
+		(stroke
+			(width 0)
+			(type default)
+		)
+	)
+	(wire
+		(pts
 			(xy 331.47 189.23) (xy 337.82 189.23)
 		)
@@
 	(wire
 		(pts
-			(xy 447.04 176.53) (xy 452.12 176.53)
-		)
-		(stroke
-			(width 0)
-			(type default)
-		)
-	)
-	(wire
-		(pts
 			(xy 92.71 364.49) (xy 92.71 370.84)
 		)
@@
 		)
 	)
+	(label "JOY_UP"
+		(at 445.77 168.91 0)
+		(effects
+			(font
+				(size 1.27 1.27)
+			)
+		)
+	)
 	(label "GND"
 		(at 57.15 69.85 0)
@@
 		)
 	)
-	(label "JOY_LEFT"
+	(label "JOY_RIGHT"
 		(at 444.5 153.67 0)
 		(effects
@@
 		)
 	)
-	(label "JOY_DOWN"
+	(label "JOY_LEFT"
 		(at 444.5 161.29 0)
 		(effects
@@
 		)
 	)
-	(label "JOY_RIGHT"
+	(label "JOY_DOWN"
 		(at 444.5 157.48 0)
 		(effects
@@
 		)
 	)
-	(label "JOY_UP"
-		(at 447.04 176.53 0)
-		(effects
-			(font
-				(size 1.27 1.27)
-			)
-		)
-	)
 	(label "+5V_LED"
 		(at 161.29 170.18 0)
@@
 		)
 	)
-	(label "JOY_DOWN"
+	(label "JOY_LEFT"
 		(at 166.37 349.25 0)
 		(effects
@@
 		)
 	)
-	(label "JOY_LEFT"
+	(label "JOY_RIGHT"
 		(at 222.25 349.25 0)
 		(effects
@@
 		)
 	)
-	(label "JOY_RIGHT"
-		(at 223.52 344.17 0)
+	(label "JOY_DOWN"
+		(at 222.25 344.17 0)
 		(effects
 			(font
@@
 	)
 	(symbol
-		(lib_id "Battery_Management:MCP73832-2-OT")
+		(lib_id "Battery_Management:MCP73832-2-MC")
 		(at 81.28 346.71 0)
 		(unit 1)
@@
 			)
 		)
-		(property "Value" "MCP73832-2-OT"
+		(property "Value" "MCP73832-2-MC"
 			(at 81.28 352.71 0)
 			(show_name no)
@@
 			)
 		)
-		(property "Footprint" "Package_TO_SOT_SMD:SOT-23-5"
+		(property "Footprint" "Package_DFN_QFN:DFN-8-1EP_3x2mm_P0.5mm_EP1.7x1.4mm"
 			(at 81.28 346.71 0)
 			(hide yes)
@@
 		(pin "5"
 		)
+		(pin "6"
+		)
+		(pin "7"
+		)
+		(pin "8"
+		)
 		(instances
